File: green-neon-indicator-board.kicad_sch (KiCad schematic)
At the start: 0 parts

Commit message: Inital schematic, component values not selected
Parts:
- added C1, C4, C5, C6, C7: UNDEF, symbol Device:C_Small
- added D1: D_Schottky, Diode_SMD:D_01005_0402Metric, symbol Device:D_Schottky
- added NE1: Green Neon Lamp, Resistor_THT:R_Axial_DIN0204_L3.6mm_D1.6mm_P2.54mm_Vertical, symbol Device:Lamp_Neon
- added Q1, Q2, Q3: Q_NMOS, symbol Device:Q_NMOS
- added R1, R10, R2, R3, R4, R5, R6, R7, R8: UNDEF, symbol Device:R_Small
- added R9: 330k, Resistor_THT:R_Axial_DIN0309_L9.0mm_D3.2mm_P15.24mm_Horizontal, symbol Device:R_Small
- added T1: Transformer_1P_1S, symbol Device:Transformer_1P_1S
- added U1: (no value), symbol Custom_Components:TI_LM5155
Connections:
- new net: Q1.D, T1.2 (AB)
- new net: D1.2 (A), T1.4 (SB)
- new net: R4.2, R5.1, U1.8 (FB)
- new net: NE1.1, R9.2
- new net: R6.1, U1.6 (COMP)
- new net: C4.1, R6.2
- new net: Q1.S, R3.1, U1.5 (CS)
- new net: C6.1, U1.2 (VCC)
- new net: R7.1, U1.10 (RT)
- new net: Q1.G, U1.3 (GATE)
- new net: C5.1, U1.9 (SS)
- new net: Q2.G, Q3.D, R10.2
- new net +150V: C7.1, D1.1 (K), R4.1, R8.1, R9.1
- new net +3.3V: C1.1, R1.1, R10.1, T1.1 (AA), U1.1 (BIAS)
- new net BOOST_EN: Q2.D, R1.2, R2.1, U1.12 (UVLO/EN/SYNC)
- new net EN_INPUT: Q3.G
- new net GND: C1.2, C4.2, C5.2, C6.2, C7.2, NE1.2, Q2.S, Q3.S, R2.2, R3.2, R5.2, R7.2, R8.2, T1.3 (SA), U1.4 (PGND), U1.7 (AGND)

Commit message: Select part numbers for enable control circuit
Parts:
- Q2, Q3: value Q_NMOS -> PJA138K; footprint (none) -> Package_TO_SOT_SMD:TSOT-23; mpn (none) -> PJA138K_R1_00001
- R10: value UNDEF -> 10k; mpn (none) -> RC0402FR-0710KL
- U1: mpn (none) -> LM5155DSSR
Changed lines of the file:
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@@
+			)
+		)
+		(property "mpn" "LM5155DSSR"
+			(at 85.09 71.12 0)
+			(hide yes)
+			(show_name no)
+			(do_not_autoplace no)
+			(effects
+				(font
+					(size 1.27 1.27)
+				)
 			)
 		)
@@
 			)
 		)
-		(property "Value" "UNDEF"
+		(property "Value" "10k"
 			(at 47.498 135.636 0)
 			(show_name no)
@@
 		)
 		(property "Description" "Resistor, small symbol"
+			(at 45.72 134.62 0)
+			(hide yes)
+			(show_name no)
+			(do_not_autoplace no)
+			(effects
+				(font
+					(size 1.27 1.27)
+				)
+			)
+		)
+		(property "mpn" "RC0402FR-0710KL"
 			(at 45.72 134.62 0)
 			(hide yes)
@@
 			)
 		)
-		(property "Value" "Q_NMOS"
+		(property "Value" "PJA138K"
 			(at 64.77 143.5099 0)
 			(show_name no)
@@
 			)
 		)
-		(property "Footprint" ""
+		(property "Footprint" "Package_TO_SOT_SMD:TSOT-23"
 			(at 63.5 139.7 0)
 			(hide yes)
@@
 		)
 		(property "Description" "N-MOSFET transistor"
+			(at 58.42 142.24 0)
+			(hide yes)
+			(show_name no)
+			(do_not_autoplace no)
+			(effects
+				(font
+					(size 1.27 1.27)
+				)
+			)
+		)
+		(property "mpn" "PJA138K_R1_00001"
+			(at 58.42 142.24 0)
+			(hide yes)
+			(show_name no)
+			(do_not_autoplace no)
+			(effects
+				(font
+					(size 1.27 1.27)
+				)
+			)
+		)
+		(property "Field6" ""
 			(at 58.42 142.24 0)
 			(hide yes)
@@
 			)
 		)
-		(property "Value" "Q_NMOS"
+		(property "Value" "PJA138K"
 			(at 49.53 149.8599 0)
 			(show_name no)
@@
 			)
 		)
-		(property "Footprint" ""
+		(property "Footprint" "Package_TO_SOT_SMD:TSOT-23"
 			(at 48.26 146.05 0)
 			(hide yes)
@@
 			(at 43.18 148.59 0)
 			(hide yes)
+			(show_name no)
+			(do_not_autoplace no)
+			(effects
+				(font
+					(size 1.27 1.27)
+				)
+			)
+		)
+		(property "mpn" "PJA138K_R1_00001"
+			(at 43.18 148.59 0)
+			(hide yes)

Commit message: Select all component values, initial layout and routing
Parts:
- removed C6: UNDEF, symbol Device:C_Small
- removed R1, R2: UNDEF, symbol Device:R_Small
- removed T1: Transformer_1P_1S, symbol Device:Transformer_1P_1S
- added C2: 100n, Capacitor_SMD:C_0402_1005Metric_Pad0.74x0.62mm_HandSolder, symbol Device:C_Small
- added J1: 1x3 THT Headers, Connector_PinHeader_2.54mm:PinHeader_1x03_P2.54mm_Vertical, symbol Connector_Generic:Conn_01x03
- added J2: JST XH Compatible, Connector_JST:JST_XH_B3B-XH-A_1x03_P2.50mm_Vertical, symbol Connector_Generic:Conn_01x03
- added R13: 100k, Resistor_SMD:R_0402_1005Metric_Pad0.72x0.64mm_HandSolder, symbol Device:R_Small
- added R6, R7: 499k, Resistor_SMD:R_0402_1005Metric_Pad0.72x0.64mm_HandSolder, symbol Device:R_Small
- added T1: WURTH_750311692, CustomLibraries:WURTH_750311692, symbol Custom_Components:WURTH_750311692
- C1: value UNDEF -> 10u; footprint (none) -> Capacitor_SMD:C_0402_1005Metric_Pad0.74x0.62mm_HandSolder
- C3: renamed from C5; value UNDEF -> 100n; footprint (none) -> Capacitor_SMD:C_0402_1005Metric_Pad0.74x0.62mm_HandSolder; mpn (none) -> GRM155R71H104KE14D
- C4: value UNDEF -> 470n; footprint (none) -> Capacitor_SMD:C_0402_1005Metric_Pad0.74x0.62mm_HandSolder; mpn (none) -> GRT155R61E474KE01D
- C5: renamed from C7; value UNDEF -> 100n; footprint (none) -> Capacitor_SMD:C_1206_3216Metric_Pad1.33x1.80mm_HandSolder; mpn (none) -> GRM31CR72D104KW03L
- D1: value D_Schottky -> US1G-E3/61T; footprint Diode_SMD:D_01005_0402Metric -> Diode_SMD:D_SMA; mpn (none) -> US1G-E3/61T
- Q1: value Q_NMOS -> IRLML0100TRPBF; footprint (none) -> Package_TO_SOT_SMD:SOT-23-3; mpn (none) -> IRLML0100TRPBF
- R10: renamed from R8; value UNDEF -> 1M; footprint (none) -> Resistor_SMD:R_0402_1005Metric_Pad0.72x0.64mm_HandSolder; mpn (none) -> RC0402FR-071ML
- R11: renamed from R9; mpn (none) -> RC0402FR-07330KL
- R12: renamed from R10; footprint (none) -> Resistor_SMD:R_0402_1005Metric_Pad0.72x0.64mm_HandSolder
- R3: renamed from R7; value UNDEF -> 110k; footprint (none) -> Resistor_SMD:R_0402_1005Metric_Pad0.72x0.64mm_HandSolder; mpn (none) -> RC0402FR-07110KL
- R4: renamed from R6; value UNDEF -> 10k; footprint (none) -> Resistor_SMD:R_0402_1005Metric_Pad0.72x0.64mm_HandSolder; mpn (none) -> RC0402FR-0710KL
- R5: renamed from R3; value UNDEF -> 0.5; footprint (none) -> Resistor_SMD:R_0402_1005Metric_Pad0.72x0.64mm_HandSolder; mpn (none) -> RL0402FR-070R5L
- R8: renamed from R4; value UNDEF -> 499k; footprint (none) -> Resistor_SMD:R_0402_1005Metric_Pad0.72x0.64mm_HandSolder; mpn (none) -> RC0402FR-07499KL
- R9: renamed from R5; value UNDEF -> 10k; footprint (none) -> Resistor_SMD:R_0402_1005Metric_Pad0.72x0.64mm_HandSolder; mpn (none) -> RC0402FR-0710KL
- U1: footprint (none) -> CustomLibraries:LM5155
Connections:
- net +3.3V is gone; now on net V_{BIAS}: C1.1, R12.1, U1.1 (BIAS)
- net +150V: now also R6.1; no longer R8.1
- net BOOST_EN: now also Q2.3 (D), R13.2; no longer Q2.D
- net EN_INPUT: now also Q3.1 (G), J1.2 (Pin_2), J2.2 (Pin_2); no longer Q3.G
- net GND: now also Q2.2 (S), Q3.2 (S), C2.2, J1.1 (Pin_1), J2.1 (Pin_1), T1.8 (SD); no longer Q2.S, Q3.S
- net at D1.2 (A): now also T1.5 (SA)
- net at R5.1, U1.5 (CS): now also Q1.2 (S); no longer Q1.S
- net V_{BIAS}: now reaches U1.2 (VCC)
- net V_{BIAS}: now also C2.1, J1.3 (Pin_3), J2.3 (Pin_3), R13.1, T1.3 (AA)
- net at U1.3 (GATE): now also Q1.1 (G); no longer Q1.G
- new net: R7.2, R8.1
- new net: Q2.1 (G), Q3.3 (D), R12.2
- new net: R6.2, R7.1
- new net: Q1.3 (D), T1.4 (AB)
- new net: T1.6 (SB), T1.7 (SC)
Other:
- note added: "For C5: Since load is so small we don't need that much filtering from the cap, and since we want this module to act like an LED replacement, the lamp may be flashed or blinked so we don't actually want to store too much charge Currently RC = 0.1s and since the lamp effectively turns off when the output drops below ~63V, the actual turn-off time will be shorter than 5RC"
- title: (none) -> Green Neon Indicator Board
- moved on the sheet: D1

Commit message: Add lcsc part number to schematic symbols, prep design for manufacturing
Parts:
- C1: footprint Capacitor_SMD:C_0402_1005Metric_Pad0.74x0.62mm_HandSolder -> Capacitor_SMD:C_0603_1608Metric_Pad1.08x0.95mm_HandSolder; manu_part_no (none) -> GRM188R61E106MA73D; mpn (none) -> C91606
- C2: manu_part_no (none) -> CC1206KKX7RABB104; mpn (none) -> C77020
- C3: manu_part_no (none) -> GRM155R71H104KE14D; mpn GRM155R71H104KE14D -> C77020
- C4: manu_part_no (none) -> GRT155R61E474KE01D; mpn GRT155R61E474KE01D -> C782164
- C5: manu_part_no (none) -> CC1206KKX7RABB104; mpn GRM31CR72D104KW03L -> C113894
- D1: manu_part_no (none) -> US1G-E3/61T; mpn US1G-E3/61T -> C82645
- J1, J2: now not fitted
- NE1: footprint Resistor_THT:R_Axial_DIN0204_L3.6mm_D1.6mm_P2.54mm_Vertical -> Connector_PinHeader_2.54mm:PinHeader_1x02_P2.54mm_Vertical; now not fitted
- Q1: manu_part_no (none) -> IRLML0100TRPBF; mpn IRLML0100TRPBF -> C53658
- Q2, Q3: manu_part_no (none) -> PJA138K_R1_00001; mpn PJA138K_R1_00001 -> C2902548
- R10: manu_part_no (none) -> RC0402FR-071ML; mpn RC0402FR-071ML -> C138033
- R11: manu_part_no (none) -> FMP200JR-52-330K; mpn RC0402FR-07330KL -> C1740085; now not fitted
- R12, R4, R9: manu_part_no (none) -> RC0402FR-0710KL; mpn RC0402FR-0710KL -> C60490
- R13: manu_part_no (none) -> RC0402FR-07100KL; mpn RC0402FR-07100KL -> C60491
- R3: manu_part_no (none) -> RC0402FR-07110KL; mpn RC0402FR-07110KL -> C138065
- R5: manu_part_no (none) -> RL0402FR-070R5L; mpn RL0402FR-070R5L -> C495757
- R6, R7, R8: manu_part_no (none) -> RC0402FR-07499KL; mpn RC0402FR-07499KL -> C137971
- T1: manu_part_no (none) -> 750311692; mpn 750311692 -> (none); now not fitted
- U1: manu_part_no (none) -> LM5155DSSR; mpn LM5155DSSR -> C778612
Connections:
- net FB: now reaches R8.2, R9.1, U1.8 (FB)
- net CS: now reaches Q1.2 (S), R5.1, U1.5 (CS)
